File: Hardware/KiCad/Thunderscope_Rev5.3/ADC_Driver.kicad_sch (KiCad schematic)
At the start: 12 parts, among them U12_4 ADA4930-1YCPZ

Commit message: Changed R136 and R137 to 4.99R, closes #433
Parts:
- R136_4, R137_4: value 10 -> 4.99; symbol Thunderscope_Rev5:RES 10 OHM 1% 1/16W 0402 -> Thunderscope_Rev5:RES 4.99 OHM 1% 1/16W 0402; MANUFACTURER PART NUMBER RC0402FR-0710RL -> RC0402FR-074R99L; SUPPLIER PART NUMBER 1 603-RC0402FR-0710RL -> 603-RC0402FR-074R99L
Changed lines of the file:
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@@
 	)
 	(symbol
-		(lib_id "Thunderscope_Rev5:RES 10 OHM 1% 1/16W 0402")
+		(lib_id "Thunderscope_Rev5:RES 4.99 OHM 1% 1/16W 0402")
 		(at 177.8 111.76 0)
 		(unit 1)
@@
 			)
 		)
-		(property "Value" "10"
+		(property "Value" "4.99"
 			(at 177.8 111.76 0)
 			(effects
@@
 			)
 		)
-		(property "Description" "10 Ohms ±1% 0.063W, 1/16W Chip Resistor 0402 (1005 Metric) Moisture Resistant Thick Film"
+		(property "Description" "4.99 Ohms ±1% 0.063W, 1/16W Chip Resistor 0402 (1005 Metric) Moisture Resistant Thick Film"
 			(at 177.8 111.76 0)
 			(effects
@@
 			)
 		)
-		(property "SUPPLIER PART NUMBER 1" "603-RC0402FR-0710RL"
+		(property "SUPPLIER PART NUMBER 1" "603-RC0402FR-074R99L"
 			(at 177.8 111.76 0)
 			(effects
@@
 			)
 		)
-		(property "MANUFACTURER PART NUMBER" "RC0402FR-0710RL"
+		(property "MANUFACTURER PART NUMBER" "RC0402FR-074R99L"
 			(at 177.8 111.76 0)
 			(effects
@@
 	)
 	(symbol
-		(lib_id "Thunderscope_Rev5:RES 10 OHM 1% 1/16W 0402")
+		(lib_id "Thunderscope_Rev5:RES 4.99 OHM 1% 1/16W 0402")
 		(at 177.8 106.68 0)
 		(unit 1)
@@
 			)
 		)
-		(property "Value" "10"
+		(property "Value" "4.99"
 			(at 177.8 106.68 0)
 			(effects
@@
 			)
 		)
-		(property "Description" "10 Ohms ±1% 0.063W, 1/16W Chip Resistor 0402 (1005 Metric) Moisture Resistant Thick Film"
+		(property "Description" "4.99 Ohms ±1% 0.063W, 1/16W Chip Resistor 0402 (1005 Metric) Moisture Resistant Thick Film"
 			(at 177.8 106.68 0)
 			(effects
@@
 			)
 		)
-		(property "SUPPLIER PART NUMBER 1" "603-RC0402FR-0710RL"
+		(property "SUPPLIER PART NUMBER 1" "603-RC0402FR-074R99L"
 			(at 177.8 106.68 0)
 			(effects
@@
 			)
 		)
-		(property "MANUFACTURER PART NUMBER" "RC0402FR-0710RL"
+		(property "MANUFACTURER PART NUMBER" "RC0402FR-074R99L"
 			(at 177.8 106.68 0)
 			(effects
