File: Hardware/KiCad/Thunderscope_Rev5.3/ACQ_FE_VREG.kicad_sch (KiCad schematic)
At the start: 66 parts, among them U13 LM27761, U14 TPS7A9101, U15 TPS7A9101, U16 TPS7A2033, U9 TPS7A2033

Commit message: Replaced TPS7A2033 LDOs with NCP161ASN330T1G, closes #434
Parts:
- U16, U9: value TPS7A2033 -> NCP161ASN330T1G; symbol Thunderscope_Rev5:IC LDO TPS7A2033 -> Thunderscope_Rev5:IC LDO NCP161ASN330T1G; MANUFACTURER Texas Instruments -> onsemi; MANUFACTURER PART NUMBER TPS7A2033PDBVR -> NCP161ASN330T1G; SUPPLIER 1 Texas Instruments -> Mouser; SUPPLIER PART NUMBER 1 TPS7A2033PDBVR -> 863-NCP161ASN330T1G
Changed lines of the file:
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@@
 	)
 	(symbol
-		(lib_id "Thunderscope_Rev5:IC LDO TPS7A2033")
+		(lib_id "Thunderscope_Rev5:IC LDO NCP161ASN330T1G")
 		(at 93.98 38.1 0)
 		(unit 1)
@@
 			)
 		)
-		(property "Value" "TPS7A2033"
+		(property "Value" "NCP161ASN330T1G"
 			(at 86.36 45.72 0)
 			(effects
@@
 			)
 		)
-		(property "Description" "Linear Voltage Regulator IC Positive Fixed 1 Output 300mA SOT-23-5"
+		(property "Description" "Linear Voltage Regulator IC Positive Fixed 1 Output 450mA SOT-23-5"
 			(at 93.98 38.1 0)
 			(effects
@@
 			)
 		)
-		(property "MANUFACTURER" "Texas Instruments"
+		(property "MANUFACTURER" "onsemi"
 			(at 78.232 27.94 0)
 			(effects
@@
 			)
 		)
-		(property "MANUFACTURER PART NUMBER" "TPS7A2033PDBVR"
+		(property "MANUFACTURER PART NUMBER" "NCP161ASN330T1G"
 			(at 78.232 27.94 0)
 			(effects
@@
 			)
 		)
-		(property "SUPPLIER 1" "Texas Instruments"
+		(property "SUPPLIER 1" "Mouser"
 			(at 78.232 27.94 0)
 			(effects
@@
 			)
 		)
-		(property "SUPPLIER PART NUMBER 1" "TPS7A2033PDBVR"
+		(property "SUPPLIER PART NUMBER 1" "863-NCP161ASN330T1G"
 			(at 78.232 27.94 0)
 			(effects
@@
 	)
 	(symbol
-		(lib_id "Thunderscope_Rev5:IC LDO TPS7A2033")
+		(lib_id "Thunderscope_Rev5:IC LDO NCP161ASN330T1G")
 		(at 83.82 175.26 0)
 		(unit 1)
@@
 			)
 		)
-		(property "Value" "TPS7A2033"
+		(property "Value" "NCP161ASN330T1G"
 			(at 76.2 182.88 0)
 			(effects
@@
 			)
 		)
-		(property "Description" "Linear Voltage Regulator IC Positive Fixed 1 Output 300mA SOT-23-5"
+		(property "Description" "Linear Voltage Regulator IC Positive Fixed 1 Output 450mA SOT-23-5"
 			(at 83.82 175.26 0)
 			(effects
@@
 			)
 		)
-		(property "MANUFACTURER" "Texas Instruments"
+		(property "MANUFACTURER" "onsemi"
 			(at 68.072 165.1 0)
 			(effects
@@
 			)
 		)
-		(property "MANUFACTURER PART NUMBER" "TPS7A2033PDBVR"
+		(property "MANUFACTURER PART NUMBER" "NCP161ASN330T1G"
 			(at 68.072 165.1 0)
 			(effects
@@
 			)
 		)
-		(property "SUPPLIER 1" "Texas Instruments"
+		(property "SUPPLIER 1" "Mouser"
 			(at 68.072 165.1 0)
 			(effects
@@
 			)
 		)
-		(property "SUPPLIER PART NUMBER 1" "TPS7A2033PDBVR"
+		(property "SUPPLIER PART NUMBER 1" "863-NCP161ASN330T1G"
 			(at 68.072 165.1 0)
 			(effects
